File: dac.kicad_sch (KiCad schematic)
At the start: 30 parts, among them J2 Conn_02x03_Odd_Even, U6 PCM5242RHBR, X1 22.5792Mhz, X2 24.576Mhz

Commit message: Replace DVDD global label with VDD power symbol
Connections:
- net DVDD renamed VDD
Changed lines of the file:
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@@
     (comment 2 "License: CERN Open Hardware Licence Version 2 - Permissive")
   )
+  (junction (at 182.88 85.09) (diameter 0) (color 0 0 0 0)
+  )
+  (junction (at 99.06 92.71) (diameter 0) (color 0 0 0 0)
+  )
+  (junction (at 85.09 90.17) (diameter 0) (color 0 0 0 0)
+  )
+  (junction (at 91.44 90.17) (diameter 0) (color 0 0 0 0)
+  )
+  (junction (at 209.55 110.49) (diameter 0) (color 0 0 0 0)
+  )
+  (junction (at 180.34 82.55) (diameter 0) (color 0 0 0 0)
+  )
+  (junction (at 96.52 125.73) (diameter 0) (color 0 0 0 0)
+  )
+  (junction (at 60.96 100.33) (diameter 0) (color 0 0 0 0)
+  )
+  (junction (at 102.87 123.19) (diameter 0) (color 0 0 0 0)
+  )
+  (junction (at 144.78 73.66) (diameter 0) (color 0 0 0 0)
+  )
+  (junction (at 214.63 73.66) (diameter 0) (color 0 0 0 0)
+  )
+  (junction (at 205.74 110.49) (diameter 0) (color 0 0 0 0)
+  )
+  (junction (at 53.34 139.7) (diameter 0) (color 0 0 0 0)
+  )
+  (junction (at 71.12 161.29) (diameter 0) (color 0 0 0 0)
+  )
+  (junction (at 175.26 110.49) (diameter 0) (color 0 0 0 0)
+  )
+  (junction (at 158.75 82.55) (diameter 0) (color 0 0 0 0)
+  )
+  (junction (at 77.47 137.16) (diameter 0) (color 0 0 0 0)
+  )
+  (junction (at 233.68 73.66) (diameter 0) (color 0 0 0 0)
+  )
+  (junction (at 182.88 110.49) (diameter 0) (color 0 0 0 0)
+  )
+  (junction (at 46.99 137.16) (diameter 0) (color 0 0 0 0)
+  )
+  (junction (at 60.96 92.71) (diameter 0) (color 0 0 0 0)
+  )
+  (junction (at 85.09 81.28) (diameter 0) (color 0 0 0 0)
+  )
+  (junction (at 53.34 161.29) (diameter 0) (color 0 0 0 0)
+  )
+  (junction (at 153.67 110.49) (diameter 0) (color 0 0 0 0)
+  )
+  (junction (at 77.47 100.33) (diameter 0) (color 0 0 0 0)
+  )
+  (junction (at 154.94 87.63) (diameter 0) (color 0 0 0 0)
+  )
+  (junction (at 90.17 118.11) (diameter 0) (color 0 0 0 0)
+  )
   (junction (at 99.06 73.66) (diameter 0) (color 0 0 0 0)
-  )
-  (junction (at 182.88 85.09) (diameter 0) (color 0 0 0 0)
-  )
-  (junction (at 99.06 92.71) (diameter 0) (color 0 0 0 0)
-  )
-  (junction (at 85.09 90.17) (diameter 0) (color 0 0 0 0)
-  )
-  (junction (at 91.44 90.17) (diameter 0) (color 0 0 0 0)
-  )
-  (junction (at 209.55 110.49) (diameter 0) (color 0 0 0 0)
-  )
-  (junction (at 180.34 82.55) (diameter 0) (color 0 0 0 0)
-  )
-  (junction (at 96.52 125.73) (diameter 0) (color 0 0 0 0)
-  )
-  (junction (at 60.96 100.33) (diameter 0) (color 0 0 0 0)
-  )
-  (junction (at 102.87 123.19) (diameter 0) (color 0 0 0 0)
-  )
-  (junction (at 144.78 73.66) (diameter 0) (color 0 0 0 0)
-  )
-  (junction (at 214.63 73.66) (diameter 0) (color 0 0 0 0)
-  )
-  (junction (at 205.74 110.49) (diameter 0) (color 0 0 0 0)
-  )
-  (junction (at 53.34 139.7) (diameter 0) (color 0 0 0 0)
-  )
-  (junction (at 71.12 161.29) (diameter 0) (color 0 0 0 0)
-  )
-  (junction (at 175.26 110.49) (diameter 0) (color 0 0 0 0)
-  )
-  (junction (at 158.75 82.55) (diameter 0) (color 0 0 0 0)
-  )
-  (junction (at 77.47 137.16) (diameter 0) (color 0 0 0 0)
-  )
-  (junction (at 233.68 73.66) (diameter 0) (color 0 0 0 0)
-  )
-  (junction (at 182.88 110.49) (diameter 0) (color 0 0 0 0)
-  )
-  (junction (at 46.99 137.16) (diameter 0) (color 0 0 0 0)
-  )
-  (junction (at 60.96 92.71) (diameter 0) (color 0 0 0 0)
-  )
-  (junction (at 85.09 81.28) (diameter 0) (color 0 0 0 0)
-  )
-  (junction (at 53.34 161.29) (diameter 0) (color 0 0 0 0)
-  )
-  (junction (at 153.67 110.49) (diameter 0) (color 0 0 0 0)
-  )
-  (junction (at 77.47 100.33) (diameter 0) (color 0 0 0 0)
-  )
-  (junction (at 154.94 87.63) (diameter 0) (color 0 0 0 0)
-  )
-  (junction (at 90.17 118.11) (diameter 0) (color 0 0 0 0)
   )
   (junction (at 71.12 139.7) (diameter 0) (color 0 0 0 0)
@@
     (stroke (width 0) (type default))
   )
-  (wire (pts (xy 95.25 73.66) (xy 99.06 73.66))
-    (stroke (width 0) (type default))
-  )
   (wire (pts (xy 190.5 77.47) (xy 224.79 77.47))
     (stroke (width 0) (type default))
@@
   (label "outr-" (at 64.77 139.7 0) (fields_autoplaced)
     (effects (font (size 1.27 1.27)) (justify left bottom))
-  )
-  (global_label "DVDD" (shape input) (at 95.25 73.66 180)
-    (effects (font (size 1.27 1.27)) (justify right))
-    (property "Intersheetrefs" "${INTERSHEET_REFS}" (at 95.25 73.66 0)
-      (effects (font (size 1.27 1.27)) hide)
-    )
   )
   (global_label "scl" (shape input) (at 151.13 123.19 0)
@@
         )
       )
+    )
+  )
+  (symbol (lib_id "power:VDD") (at 99.06 73.66 0) (unit 1)
+    (in_bom yes) (on_board yes) (dnp no) (fields_autoplaced)
+    (property "Reference" "#PWR022" (at 99.06 77.47 0)
+      (effects (font (size 1.27 1.27)) hide)
+    )
+    (property "Value" "VDD" (at 99.06 68.58 0)
+      (effects (font (size 1.27 1.27)))
+    )
+    (property "Footprint" "" (at 99.06 73.66 0)
+      (effects (font (size 1.27 1.27)) hide)
+    )
+    (property "Datasheet" "" (at 99.06 73.66 0)
+      (effects (font (size 1.27 1.27)) hide)
+    )
+    (pin "1")
+    (instances
+      (project "pedalboard-soundcard"
+        (path "/257597c6-fbef-4478-b0f4-968f2d6f1866/c0100554-f979-4e8d-b08c-e48cc1e12bdc"
+          (reference "#PWR022") (unit 1)
+        )
+      )
