File: dac.kicad_sch (KiCad schematic)
At the start: 33 parts, among them J2 Conn_02x03_Odd_Even, J5 Audio_Jack, U6 PCM5242RHBR, X1 22.5792Mhz, X2 24.576Mhz

Commit message: Add first pnp job
Parts:
- C20, C28, C29, C32: value 100nF25V -> 100n
- C21, C22, C25, C26: value 2,2nF50V -> 2n2
- C23, C24, C27, C30, C31: value 1uF16V -> 1u
- D2: value LED -> red
- X1: value 22.5792Mhz -> 22.5792M
- X2: value 24.576Mhz -> 24.576M
Changed lines of the file:
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@@
 			)
 		)
-		(property "Value" "1uF16V"
+		(property "Value" "1u"
 			(at 69.85 82.55 0)
 			(effects
@@
 			)
 		)
-		(property "Value" "100nF25V"
+		(property "Value" "100n"
 			(at 45.339 95.377 0)
 			(effects
@@
 			)
 		)
-		(property "Value" "1uF16V"
+		(property "Value" "1u"
 			(at 96.139 99.187 0)
 			(effects
@@
 			)
 		)
-		(property "Value" "LED"
+		(property "Value" "red"
 			(at 165.2778 121.285 0)
 			(effects
@@
 			)
 		)
-		(property "Value" "100nF25V"
+		(property "Value" "100n"
 			(at 80.01 125.73 0)
 			(effects
@@
 			)
 		)
-		(property "Value" "100nF25V"
+		(property "Value" "100n"
 			(at 95.25 82.55 0)
 			(effects
@@
 			)
 		)
-		(property "Value" "2,2nF50V"
+		(property "Value" "2n2"
 			(at 66.04 153.67 0)
 			(effects
@@
 			)
 		)
-		(property "Value" "24.576Mhz"
+		(property "Value" "24.576M"
 			(at 223.52 119.38 0)
 			(effects
@@
 			)
 		)
-		(property "Value" "2,2nF50V"
+		(property "Value" "2n2"
 			(at 38.1 153.67 0)
 			(effects
@@
 			)
 		)
-		(property "Value" "100nF25V"
+		(property "Value" "100n"
 			(at 241.681 82.423 0)
 			(effects
@@
 			)
 		)
-		(property "Value" "1uF16V"
+		(property "Value" "1u"
 			(at 58.039 95.377 0)
 			(effects
@@
 			)
 		)
-		(property "Value" "1uF16V"
+		(property "Value" "1u"
 			(at 102.87 125.73 0)
 			(effects
@@
 			)
 		)
-		(property "Value" "1uF16V"
+		(property "Value" "1u"
 			(at 90.17 104.14 90)
 			(effects
@@
 			)
 		)
-		(property "Value" "22.5792Mhz"
+		(property "Value" "22.5792M"
 			(at 223.52 85.09 0)
 			(effects
@@
 			)
 		)
-		(property "Value" "2,2nF50V"
+		(property "Value" "2n2"
 			(at 78.74 153.67 0)
 			(effects
@@
 			)
 		)
-		(property "Value" "2,2nF50V"
+		(property "Value" "2n2"
 			(at 50.8 153.67 0)
 			(effects

Commit message: Align LED value with other projects
Parts:
- D2: value red -> LED_R
Changed lines of the file:
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@@
 			)
 		)
-		(property "Value" "red"
+		(property "Value" "LED_R"
 			(at 165.2778 121.285 0)
 			(effects

Commit message: Update the oscilator part definitions
Parts:
- X1: Supplier https://www.digikey.ch/de/products/detail/abracon-llc/ASV-2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 -> https://www.digikey.ch/en/products/detail/kyocera-avx/KC201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
- X2: Supplier https://www.digikey.ch/de/products/detail/abracon-llc/ASDMB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 -> https://www.digikey.ch/en/products/detail/kyocera-avx/KC201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
Changed lines of the file:
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@@
 			)
 		)
-		(property "Datasheet" "https://abracon.com/Oscillators/ASCO.pdf"
+		(property "Datasheet" "https://media.digikey.com/pdf/Data%20Sheets/Kyocera%20International/Z_Series_X_Type.pdf"
 			(at 208.915 112.395 0)
 			(effects
@@
 			)
 		)
-		(property "Supplier" "https://www.digikey.ch/de/products/detail/abracon-llc/ASDMB-24-576MHZ-LC-T/2809941"
+		(property "Supplier" "https://www.digikey.ch/en/products/detail/kyocera-avx/KC2016Z24-5760C1KX00/11610181"
 			(at 214.63 115.57 0)
 			(effects
@@
 			)
 		)
-		(property "Datasheet" "https://abracon.com/Oscillators/ASCO.pdf"
+		(property "Datasheet" "https://media.digikey.com/pdf/Data%20Sheets/Kyocera%20International/Z_Series_X_Type.pdf"
 			(at 208.915 78.105 0)
 			(effects
@@
 			)
 		)
-		(property "Supplier" "https://www.digikey.ch/de/products/detail/abracon-llc/ASV-22-5792MHZ-LR-T/15995980"
+		(property "Supplier" "https://www.digikey.ch/en/products/detail/kyocera-avx/KC2016Z22-5792C1KX00/11610237"
 			(at 214.63 81.28 0)
 			(effects
