File: pedalboard-soundcard.kicad_sch (KiCad schematic)
At the start: 30 parts, among them J1 RPi_GPIO, T1 Tab, T2 Tab, T3 Tab, T4 Tab, U1 AT24CS01-STUM, U2 NCP163, U3 NCP163, U5 NCP163

Commit message: Add first pnp job
Parts:
- C1: value 100nF25V -> 100n
- C10, C12, C5, C6, C8, C9: value 10uF16V -> 10u
Changed lines of the file:
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@@
 			)
 		)
-		(property "Value" "10uF16V"
+		(property "Value" "10u"
 			(at 135.89 66.04 0)
 			(effects
@@
 			)
 		)
-		(property "Value" "10uF16V"
+		(property "Value" "10u"
 			(at 255.27 66.04 0)
 			(effects
@@
 			)
 		)
-		(property "Value" "10uF16V"
+		(property "Value" "10u"
 			(at 165.1 66.04 0)
 			(effects
@@
 			)
 		)
-		(property "Value" "10uF16V"
+		(property "Value" "10u"
 			(at 208.28 66.04 0)
 			(effects
@@
 			)
 		)
-		(property "Value" "10uF16V"
+		(property "Value" "10u"
 			(at 233.68 66.04 0)
 			(effects
@@
 			)
 		)
-		(property "Value" "10uF16V"
+		(property "Value" "10u"
 			(at 180.34 67.31 0)
 			(effects
@@
 			)
 		)
-		(property "Value" "100nF25V"
+		(property "Value" "100n"
 			(at 28.829 115.697 0)
 			(effects
