File: adc.kicad_sch (KiCad schematic)
At the start: 28 parts, among them J3 Conn_02x03_Odd_Even, J4 Audio_Jack, U4 PCM1863DBT

Commit message: Improve bom
Parts:
- C33, C34: Supplier https://www.digikey.ch/de/products/detail/samsung-electro-m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 -> https://www.digikey.ch/en/products/detail/panasonic-electro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
Changed lines of the file:
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@@
 			)
 		)
-		(property "Datasheet" "https://www.samsungsem.com/resources/file/global/support/product_catalog/MLCC.pdf"
+		(property "Datasheet" "https://industrial.panasonic.com/ww/products/pt/film-cap-electroequip/models/ECHU1C103JX5"
 			(at 180.34 104.14 0)
 			(effects
@@
 			)
 		)
-		(property "Supplier" "https://www.digikey.ch/de/products/detail/samsung-electro-mechanics/CL21B104KBCNNNC/3886661"
+		(property "Supplier" "https://www.digikey.ch/en/products/detail/panasonic-electronic-components/ECH-U1C103JX5/353645"
 			(at 180.34 104.14 0)
 			(effects
@@
 			)
 		)
-		(property "Datasheet" "https://www.samsungsem.com/resources/file/global/support/product_catalog/MLCC.pdf"
+		(property "Datasheet" "https://industrial.panasonic.com/ww/products/pt/film-cap-electroequip/models/ECHU1C103JX5"
 			(at 149.86 104.14 0)
 			(effects
@@
 			)
 		)
-		(property "Supplier" "https://www.digikey.ch/de/products/detail/samsung-electro-mechanics/CL21B104KBCNNNC/3886661"
+		(property "Supplier" "https://www.digikey.ch/en/products/detail/panasonic-electronic-components/ECH-U1C103JX5/353645"
 			(at 149.86 104.14 0)
 			(effects

Commit message: Add first pnp job
Parts:
- C11, C14, C16, C19: value 100nF25V -> 100n
- C13, C17, C18: value 1uF16V -> 1u
- C15, C2, C3, C4, C7: value 10uF16V -> 10u
- C33, C34: value 10nF -> 10n_film
- D1: value LED -> red
Changed lines of the file:
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@@
 			)
 		)
-		(property "Value" "10uF16V"
+		(property "Value" "10u"
 			(at 161.671 124.333 0)
 			(effects
@@
 			)
 		)
-		(property "Value" "10uF16V"
+		(property "Value" "10u"
 			(at 145.161 124.333 0)
 			(effects
@@
 			)
 		)
-		(property "Value" "1uF16V"
+		(property "Value" "1u"
 			(at 241.3 48.26 0)
 			(effects
@@
 			)
 		)
-		(property "Value" "1uF16V"
+		(property "Value" "1u"
 			(at 229.87 74.93 0)
 			(effects
@@
 			)
 		)
-		(property "Value" "10nF"
+		(property "Value" "10n_film"
 			(at 183.134 97.79 0)
 			(effects
@@
 			)
 		)
-		(property "Value" "1uF16V"
+		(property "Value" "1u"
 			(at 209.55 85.09 0)
 			(effects
@@
 			)
 		)
-		(property "Value" "10uF16V"
+		(property "Value" "10u"
 			(at 187.96 60.96 0)
 			(effects
@@
 			)
 		)
-		(property "Value" "10nF"
+		(property "Value" "10n_film"
 			(at 152.654 97.79 0)
 			(effects
@@
 			)
 		)
-		(property "Value" "100nF25V"
+		(property "Value" "100n"
 			(at 165.1 60.96 0)
 			(effects
@@
 			)
 		)
-		(property "Value" "100nF25V"
+		(property "Value" "100n"
 			(at 193.04 85.09 0)
 			(effects
@@
 			)
 		)
-		(property "Value" "100nF25V"
+		(property "Value" "100n"
 			(at 242.57 74.93 0)
 			(effects
@@
 			)
 		)
-		(property "Value" "LED"
+		(property "Value" "red"
 			(at 43.18 58.42 0)
 			(effects
@@
 			)
 		)
-		(property "Value" "100nF25V"
+		(property "Value" "100n"
 			(at 228.6 48.26 0)
 			(effects
@@
 			)
 		)
-		(property "Value" "10uF16V"
+		(property "Value" "10u"
 			(at 192.151 124.333 0)
 			(effects
@@
 			)
 		)
-		(property "Value" "10uF16V"
+		(property "Value" "10u"
 			(at 175.641 124.333 0)
 			(effects

Commit message: Align LED value with other projects
Parts:
- D1: value red -> LED_R
Changed lines of the file:
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@@
 			)
 		)
-		(property "Value" "red"
+		(property "Value" "LED_R"
 			(at 43.18 58.42 0)
 			(effects
