File: latest/panel/pedalboard-soundcard-panel.kicad_pcb (KiCad board)
At the start: 2 copper layers, 147 x 115 mm, 408 parts, among them J1 RPi_GPIO, J2 Conn_02x03_Odd_Even, J3 Conn_02x03_Odd_Even, J4 Audio_Jack, J5 Audio_Jack, U1 AT24CS01-STUM, U2 NCP163, U3 NCP163, U4 PCM1863DBT, U5 NCP163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

Commit message: Deploying to gh-pages from @ pedalboard/pedalboard-soundcard@95a273a64299cf2b04a6bcd4cb679e8c689c30cb 🚀
Other:
- board text added: "Open Pedalboard Soundcard github.com/pedalboard PCB: 1.0.1-RC 95a273a"
- board text removed: "Open Pedalboard Soundcard github.com/pedalboard PCB: 1.0.1-RC cfda140"

Commit message: Deploying to gh-pages from @ pedalboard/pedalboard-soundcard@80062617507ac7933be18997dff7502358ed753e 🚀
Other:
- board text added: "Open Pedalboard Soundcard github.com/pedalboard PCB: 1.0.1-RC 8006261"
- board text removed: "Open Pedalboard Soundcard github.com/pedalboard PCB: 1.0.1-RC 95a273a"

Commit message: Deploying to gh-pages from @ pedalboard/pedalboard-soundcard@b651fcc4d9002e7f3acbf86250d468447af45510 🚀
Other:
- board text added: "Open Pedalboard Soundcard github.com/pedalboard PCB: 1.0.1-RC b651fcc"
- board text removed: "Open Pedalboard Soundcard github.com/pedalboard PCB: 1.0.1-RC 8006261"
