File: latest/panel/pedalboard-soundcard-panel.kicad_pcb (KiCad board)
At the start: 2 copper layers, 147 x 115 mm, 408 parts, among them J1 RPi_GPIO, J2 Conn_02x03_Odd_Even, J3 Conn_02x03_Odd_Even, J4 Audio_Jack, J5 Audio_Jack, U1 AT24CS01-STUM, U2 NCP163, U3 NCP163, U4 PCM1863DBT, U5 NCP163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

Commit message: Deploying to gh-pages from @ pedalboard/pedalboard-soundcard@31afb6017ae6b522b8181885fa29b64f5e88adff 🚀
Other:
- board text added: "Open Pedalboard Soundcard github.com/pedalboard PCB: 1.0.1-RC 31afb60"
- board text removed: "Open Pedalboard Soundcard github.com/pedalboard PCB: 1.0.1-RC b651fcc"

Commit message: Deploying to gh-pages from @ pedalboard/pedalboard-soundcard@121d40d3377e59054d80a3f7628d9cd9ecaca75b 🚀
Other:
- board text added: "Open Pedalboard Soundcard github.com/pedalboard PCB: 1.0.1-RC 121d40d"
- board text removed: "Open Pedalboard Soundcard github.com/pedalboard PCB: 1.0.1-RC 31afb60"

Commit message: Deploying to gh-pages from @ pedalboard/pedalboard-soundcard@14fb67eb2d38b9647849726f6b280fd76ecebb48 🚀
Other:
- board text added: "Open Pedalboard Soundcard github.com/pedalboard PCB: 1.0.1-RC 14fb67e"
- board text removed: "Open Pedalboard Soundcard github.com/pedalboard PCB: 1.0.1-RC 121d40d"
