File: latest/panel/pedalboard-soundcard-panel.kicad_pcb (KiCad board)
At the start: 2 copper layers, 147 x 115 mm, 408 parts, among them J1 RPi_GPIO, J2 Conn_02x03_Odd_Even, J3 Conn_02x03_Odd_Even, J4 Audio_Jack, J5 Audio_Jack, U1 AT24CS01-STUM, U2 NCP163, U3 NCP163, U4 PCM1863DBT, U5 NCP163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

Commit message: Deploying to gh-pages from @ pedalboard/pedalboard-soundcard@77f580b22c44a5be41898fd2f4921ac181a39a88 🚀
Other:
- board text added: "Open Pedalboard Soundcard github.com/pedalboard PCB: 1.0.1-RC 77f580b"
- board text removed: "Open Pedalboard Soundcard github.com/pedalboard PCB: 1.0.1-RC 0fbefd4"

Commit message: Deploying to gh-pages from @ pedalboard/pedalboard-soundcard@b920d0f60fa750fc830212c47e7f0d8dba3abd35 🚀
Other:
- board text added: "Open Pedalboard Soundcard github.com/pedalboard PCB: 1.0.1-RC b920d0f"
- board text removed: "Open Pedalboard Soundcard github.com/pedalboard PCB: 1.0.1-RC 77f580b"

Commit message: Deploying to gh-pages from @ pedalboard/pedalboard-soundcard@dc562330052bb9dca7300b94083724d9ba66bf31 🚀
Other:
- board text added: "Open Pedalboard Soundcard github.com/pedalboard PCB: 1.0.1-RC dc56233"
- board text removed: "Open Pedalboard Soundcard github.com/pedalboard PCB: 1.0.1-RC b920d0f"
